File: sch/quiz-sch.sch (KiCad schematic (older format))
At the start: 71 parts, among them IC1 74HC4050, J1 USB_B_Micro, J2 AVR ISP, Q1 BC817, Q2 BC817, SW1 MUTE_SW, SW2 PROG_SW, SW3 SW_UP, SW4 SW_DOWN, SW5 SW_LEFT, SW6 SW_RIGHT, SW7 SW_ENTER, SW8 SW_MENU, U1 MCP73831-2-OT, U2 ATmega328P-AU, U3 TPS61092, U4 LD1117S33TR_SOT223, U5 74HCT4051, U6 FT232RL, U7 NOKIA5510, U8 24LC16BT-I_OT, Y1 16MHz

Commit message: Added PDF of schematic
Parts:
- added R25: 100K, Resistors_SMD:R_0805_HandSoldering, symbol Device:R_Small
- IC1: symbol 7400-ic:74HC4050 -> quiz-sch-rescue:74HC4050-7400-ic
- U2: symbol MCU_Microchip_ATmega:ATmega328P-AU -> quiz-sch-rescue:ATmega328P-AU-MCU_Microchip_ATmega
- U7: symbol guff:NOKIA5510 -> quiz-sch-rescue:NOKIA5510-guff
- U8: symbol guff:24LC16BT-I_OT -> quiz-sch-rescue:24LC16BT-I_OT-guff
Connections:
- net labels added: +5V
- net labels removed: 5V
- wire segments 336 -> 341
Other:
- moved on the sheet: C11, C12, R5, U4
